File: TexasInstruments-TI994A-32KB/kicad/sidecar.kicad_sch (KiCad schematic)
At the start: 10 parts, among them J1 AVR-JTAG-10, J2 Conn_02x22_Odd_Even, U1 CY62256-70PC, U2 ATF1502AS

Commit message: restored sop memory
Parts:
- J1: footprint Connector_PinHeader_2.54mm:PinHeader_2x05_P2.54mm_Vertical -> (none)
- U1: footprint Package_SO:TSOP-I-28_11.8x8mm_P0.55mm -> Package_SO:SOIC-28W_7.5x17.9mm_P1.27mm
Connections:
- net GND: no longer J1.10 (GND), J1.2 (GND)
- net TCK: no longer J1.1 (TCK)
- net TDI: no longer J1.9 (TDI)
- net TDO: no longer J1.3 (TDO)
- net TMS: no longer J1.5 (TMS)
- net VCC: no longer J1.4 (VREF), J1.7 (VCC)
- new net: J1.10 (GND), J1.2 (GND)
- no-connect marks 5 -> 18
Other:
- title: TI-99/4A 32KB Memory Expansion -> BackBit C64
